File: Ohmmeter.kicad_sch (KiCad schematic)
At the start: 0 parts

Commit message: add: charger circuit schematic complete
Parts:
- added C1, C2: 1uF, symbol Device:C_Small
- added D1: LED_Small, symbol Device:LED_Small
- added IC1: BQ21040DBVR, SOT95P280X145-6N, symbol SamacSys_Parts:BQ21040DBVR
- added IC2: BQ29737DSER, SON50P150X150X80-6N, symbol SamacSys_Parts:BQ29737DSER
- added J1: PowerIn, symbol Connector:USB_C_Receptacle_PowerOnly_6P
- added J2: Battery, Connector_JST:JST_EH_B2B-EH-A_1x02_P2.50mm_Vertical, symbol PCM_SL_Connectors:JST_02
- added R1: 10K, symbol Device:R_Small_US
- added R2: 2K, symbol Device:R_Small_US
- added R3: R_Small_US, symbol Device:R_Small_US
Connections:
- new net: IC1.1 (TS), R1.1
- new net: IC1.4 (ISET), R2.1
- new net: D1.2 (A), R3.2
- new net GND: C1.2, C2.2, IC1.5 (GND), J1.A12 (GND), J1.B12 (GND), J1.S1 (SHIELD), J2.2, R1.2, R2.2
- new net VBat: C2.1, IC1.2 (VOUT), J2.1
- new net VOUT: R3.1
- new net Vbus: J1.A9 (VBUS), J1.B9 (VBUS)
- new net Vbus_f: C1.1, IC1.6 (VIN)
- new net ~{CHG}: D1.1 (K), IC1.3 (~{CHG})
- no-connect marks 0 -> 2

Commit message: feat: battery protection
Parts:
- added C3: 0.1uF, symbol Device:C_Small
- added Q1, Q2: CSD16406Q3, DQG_VSON-CLIP, symbol SamacSys_Parts:CSD16406Q3
- added R4: 2K, symbol Device:R_Small_US
- added R5: 330R, symbol Device:R_Small_US
- added R6, R7: 5M, symbol Device:R_Small_US
Connections:
- net GND: now also IC2.4 (VSS), C3.2, Q1.5 (D_1), Q1.6 (D_2), Q1.7 (D_3), Q1.8 (D_4), Q2.5 (D_1), Q2.6 (D_2), Q2.7 (D_3), Q2.8 (D_4), R4.2
- net at IC2.2 (COUT): now also Q1.4 (G), R7.2
- net at IC2.3 (DOUT): now also Q2.4 (G), R6.1
- net at IC2.5 (BAT): now also C3.1, R5.2
- net at IC2.6 (V-): now also R4.1
- net VBat renamed Pack+
- net Pack+: now also R5.1
- new net: Q1.1 (S_1), Q1.2 (S_2), Q1.3 (S_3), R7.1
- new net: Q2.1 (S_1), Q2.2 (S_2), Q2.3 (S_3), R6.2
Other:
- moved on the sheet: IC2
